Commit message: Fix camera frame and head yaw for HRI practice

File: rb1_description/robots/rb1_robot.urdf.xacro (robot description, xacro)
@@ -55,15 +55,4 @@
       <state_interface name="effort"/>
     </joint>
-    <joint name="j1_head">
-      <command_interface name="position">
-        <param name="min">-3.14159</param>
-        <param name="max">3.14159</param>
-      </command_interface>
-      <state_interface name="position">
-        <param name="initial_value">0.0</param>
-      </state_interface>
-      <state_interface name="velocity"/>
-      <state_interface name="effort"/>
-    </joint>
     <joint name="j2_head">
       <command_interface name="position">

File: rb1_description/urdf/sensors/asus_xtion.urdf.xacro (robot description, xacro)
@@ -42,5 +42,5 @@
     </link>
     <joint name="camera_frame_joint" type="fixed">
-      <origin xyz="0 0 0" rpy="-${math_pi_over_2} 0 -${math_pi_over_2}" />
+      <origin xyz="0.000 0.000 0.000" rpy="0 0 0" />
       <parent link="${prefix}_link" />
       <child link="camera_frame" />

File: rb1_description/urdf/torsos/torso_3dof.urdf.xacro (robot description, xacro)
@@ -145,11 +145,8 @@
     </collision>
   </link>
-  <joint name="j1_head" type="revolute">
+  <joint name="j1_head" type="fixed">
     <origin xyz="0.010 0.0 0.940" rpy="0 0 0" />
     <parent link="torso_front_link" />
     <child link="head_link" />
-    <axis xyz="0 0 1" />
-    <limit effort="${joint_effort_limit}" velocity="${joint_velocity_limit}" upper="${PI/2}" lower="${-PI/2}"/>
-    <dynamics damping="${joint_damping}" friction="${joint_friction}"/>
   </joint>
   <transmission name="j1_head_trans">

Commit message: feat: head up-down fixed

File: rb1_description/robots/rb1_robot.urdf.xacro (robot description, xacro)
@@ -55,15 +55,4 @@
       <state_interface name="effort"/>
     </joint>
-    <joint name="j2_head">
-      <command_interface name="position">
-        <param name="min">-3.14159</param>
-        <param name="max">3.14159</param>
-      </command_interface>
-      <state_interface name="position">
-        <param name="initial_value">0.0</param>
-      </state_interface>
-      <state_interface name="velocity"/>
-      <state_interface name="effort"/>
-    </joint>
   </ros2_control>
   <gazebo>

File: rb1_description/urdf/torsos/torso_3dof.urdf.xacro (robot description, xacro)
@@ -25,6 +25,4 @@
   <xacro:property name="j1_head_mechanical_reduction" value="320.0"/>
   <xacro:property name="j1_head_motor_torque_constant" value="1.0"/>
-  <xacro:property name="j2_head_mechanical_reduction" value="320.0"/>
-  <xacro:property name="j2_head_motor_torque_constant" value="1.0"/>
   <xacro:macro name="torso_3dof" params="name hq">
   <!-- parameters -->
@@ -189,23 +187,9 @@
     </collision>
   </link>
-  <joint name="j2_head"    type="revolute">
+  <joint name="j2_head"    type="fixed">
     <origin xyz="0.105 0.0 0.0" rpy="0 0 0" />
     <parent link="head_link" />
     <child link="eyes_link" />
-    <!-- check --> <!-- axis xyz="0 1 0" / -->
-    <axis xyz="0 -1 0"/>
-    <limit effort="${joint_effort_limit}" velocity="${joint_velocity_limit}" upper="${PI/4}" lower="${-PI/4}"/>
-    <dynamics damping="${joint_damping}" friction="${joint_friction}"/>
-  </joint>
-  <transmission name="j2_head_trans">
-    <type>transmission_interface/SimpleTransmission</type>
-    <joint name="j2_head">
-      <hardwareInterface>hardware_interface/EffortJointInterface</hardwareInterface>
-    </joint>
-    <actuator name="j2_head_motor">
-      <mechanicalReduction>${j2_head_mechanical_reduction}</mechanicalReduction>
-      <motorTorqueConstant>${j2_head_motor_torque_constant}</motorTorqueConstant>
-    </actuator>
-  </transmission>
+  </joint>
   <joint name="torso_arm_joint" type="fixed">
     <origin xyz="-0.0127 0 0.251" rpy="0.0 0.0 0.0" />
